File: packages/chip/board/kicad/e1-phone/schematic/compute.kicad_sch (KiCad schematic)
At the start: 0 parts

Commit message: chip(e1-phone): re-render exploded animation with corrected framing + lighting + EGL chunking
Visual self-review of the previous render exposed three defects that this commit closes:

- Camera was at radius 220 mm with 35deg yfov; phone is ~155 mm tall with parts that fly ~150 mm outward at peak explode, so the camera was effectively inside the explosion bubble. Bumped radius to 500 mm and narrowed yfov to 28deg; tilt to 15deg.
- Lights were camera-anchored, so the back of the orange shell went muddy during the 360deg orbit. Switched to world-anchored 3-point lighting.
- pyrender EGL leaked GPU memory and consistently died around frame ~150. Recreating OffscreenRenderer every 30 frames keeps the full 360-frame render stable.

Re-render output (all confirmed by reading 4 keyframes):
- e1-phone-exploded.mp4: 1920x1080, 30 fps, 12 s, h264/yuv420p, 897 KB
- e1-phone-exploded.glb: 98 nodes, 97 meshes, 3 clips (explode/reassemble/turntable), 183 KB
- e1-phone-exploded-frames/: 360 sequential frames + 24 keyframes at 0.5 s

Also restores the chip e1-phone artifacts (mechanical, board, supplier-pinouts, generator scripts) that an out-of-band git reset to origin/develop wiped between my previous commits ae3f83e9e7 / bd0a350198 and the current HEAD.

Co-Authored-By: Claude Opus 4.7 (1M context) <noreply@anthropic.com>
Parts:
- added C100, C101, C102, C103, C104, C105, C106, C107: 100nF, Capacitor_SMD:C_0402_1005Metric, symbol Device:C
- added U1: E1_PhoneSoC_BGA256, Package_BGA:BGA-256_14x14mm_Layout16x16_P0.8mm, symbol e1_phone:E1_PhoneSoC_BGA256
- added U2: LPDDR5X_x32_8GiB, Package_BGA:BGA-200_LPDDR5X_x32_planning, symbol e1_phone:LPDDR5X_x32
Connections:
- new net BOOT_MODE0: U1.17 (DRAM_DQ16)
- new net BOOT_MODE1: U1.16 (DRAM_DQ15)
- new net BOOT_MODE2: U1.15 (DRAM_DQ14)
- new net CHG_I2C_SCL: U1.27 (DRAM_DQ26)
- new net CHG_I2C_SDA: U1.26 (DRAM_DQ25)
- new net CHG_IRQ_N: U1.22 (DRAM_DQ21)
- new net DISP_BL_EN: U1.60 (MIPI_DSI_D0_N)
- new net DISP_BL_PWM: U1.59 (MIPI_DSI_D0_P)
- new net DISP_RESET_N: U1.62 (MIPI_DSI_D1_N)
- new net DISP_TE: U1.61 (MIPI_DSI_D1_P)
- new net DRAM_CA0: U1.84 (MIPI_CSI1_D0_N), U2.7 (DQ6)
- new net DRAM_CA1: U1.83 (MIPI_CSI1_D0_P), U2.6 (DQ5)
- new net DRAM_CA2: U1.82 (MIPI_CSI1_CLK_N), U2.5 (DQ4)
- new net DRAM_CA3: U1.81 (MIPI_CSI1_CLK_P), U2.4 (DQ3)
- new net DRAM_CA4: U1.80 (MIPI_CSI0_D3_N), U2.3 (DQ2)
- new net DRAM_CA5: U1.79 (MIPI_CSI0_D3_P), U2.2 (DQ1)
- new net DRAM_CKE: U1.76 (MIPI_CSI0_D1_N), U2.101 (VSS)
- new net DRAM_CK_C: U1.77 (MIPI_CSI0_D2_P), U2.102 (VSS)
- new net DRAM_CK_T: U1.78 (MIPI_CSI0_D2_N), U2.1 (DQ0)
- new net DRAM_CS: U1.75 (MIPI_CSI0_D1_P), U2.100 (VSS)
- new net DRAM_DM0: U1.88 (USB_DN), U2.11 (DQ10)
- new net DRAM_DM1: U1.87 (USB_DP), U2.10 (DQ9)
- new net DRAM_DM2: U1.86 (MIPI_CSI1_D1_N), U2.9 (DQ8)
- new net DRAM_DM3: U1.85 (MIPI_CSI1_D1_P), U2.8 (DQ7)
- new net DRAM_DQ0: U1.128 (NC128), U2.51 (CK_T)
- new net DRAM_DQ1: U1.127 (NC127), U2.50 (CA5)
- new net DRAM_DQ10: U1.118 (VDD_NPU), U2.41 (DM0)
- new net DRAM_DQ11: U1.117 (VDD_GPU), U2.40 (DQS_C3)
- new net DRAM_DQ12: U1.116 (VDD_CORE), U2.39 (DQS_T3)
- new net DRAM_DQ13: U1.115 (OSC_CLK_IN), U2.38 (DQS_C2)
- new net DRAM_DQ14: U1.114 (BOOT_MODE2), U2.37 (DQS_T2)
- new net DRAM_DQ15: U1.113 (BOOT_MODE1), U2.36 (DQS_C1)
- new net DRAM_DQ16: U1.112 (BOOT_MODE0), U2.35 (DQS_T1)
- new net DRAM_DQ17: U1.111 (VOL_DOWN_N), U2.34 (DQS_C0)
- new net DRAM_DQ18: U1.110 (VOL_UP_N), U2.33 (DQS_T0)
- new net DRAM_DQ19: U1.109 (PWR_KEY_N), U2.32 (DQ31)
- new net DRAM_DQ2: U1.126 (NC126), U2.49 (CA4)
- new net DRAM_DQ20: U1.108 (SOC_RESET_N), U2.31 (DQ30)
- new net DRAM_DQ21: U1.107 (CHG_IRQ_N), U2.30 (DQ29)
- new net DRAM_DQ22: U1.106 (USBPD_IRQ_N), U2.29 (DQ28)
- new net DRAM_DQ23: U1.105 (PMIC_RESET_N), U2.28 (DQ27)
- new net DRAM_DQ24: U1.104 (PMIC_IRQ_N), U2.27 (DQ26)
- new net DRAM_DQ25: U1.103 (CHG_I2C_SDA), U2.26 (DQ25)
- new net DRAM_DQ26: U1.102 (CHG_I2C_SCL), U2.25 (DQ24)
- new net DRAM_DQ27: U1.101 (USBPD_I2C_SDA), U2.24 (DQ23)
- new net DRAM_DQ28: U1.100 (USBPD_I2C_SCL), U2.23 (DQ22)
- new net DRAM_DQ29: U1.99 (PMIC_I2C_SDA), U2.22 (DQ21)
- new net DRAM_DQ3: U1.125 (NC125), U2.48 (CA3)
- new net DRAM_DQ30: U1.98 (PMIC_I2C_SCL), U2.21 (DQ20)
- new net DRAM_DQ31: U1.97 (SPMI_SDATA), U2.20 (DQ19)
- new net DRAM_DQ4: U1.124 (VSS), U2.47 (CA2)
- new net DRAM_DQ5: U1.123 (VDD2_LPDDR), U2.46 (CA1)
- new net DRAM_DQ6: U1.122 (VDDQ_LPDDR), U2.45 (CA0)
- new net DRAM_DQ7: U1.121 (VDD_PLL), U2.44 (DM3)
- new net DRAM_DQ8: U1.120 (VDD_IO33), U2.43 (DM2)
- new net DRAM_DQ9: U1.119 (VDD_IO18), U2.42 (DM1)
- new net DRAM_DQS_C0: U1.95 (UART_RX), U2.18 (DQ17)
- new net DRAM_DQS_C1: U1.93 (JTAG_TRST_N), U2.16 (DQ15)
- new net DRAM_DQS_C2: U1.91 (JTAG_TDI), U2.14 (DQ13)
- new net DRAM_DQS_C3: U1.89 (JTAG_TCK), U2.12 (DQ11)
- new net DRAM_DQS_T0: U1.96 (SPMI_SCLK), U2.19 (DQ18)
- new net DRAM_DQS_T1: U1.94 (UART_TX), U2.17 (DQ16)
- new net DRAM_DQS_T2: U1.92 (JTAG_TDO), U2.15 (DQ14)
- new net DRAM_DQS_T3: U1.90 (JTAG_TMS), U2.13 (DQ12)
- new net DRAM_RESET_N: U1.74 (MIPI_CSI0_D0_N), U2.99 (VSS)
- new net DRAM_ZQ: U1.73 (MIPI_CSI0_D0_P), U2.98 (VSS)
- new net GND: U1.5 (DRAM_DQ4), U2.52 (CK_C), U2.53 (CKE), U2.54 (CS), U2.55 (RESET_N), U2.56 (ZQ), U2.57 (VDDQ), U2.58 (VDDQ), U2.59 (VDDQ), U2.60 (VDDQ), U2.61 (VDD2), U2.62 (VDD2), U2.63 (VDD2), U2.64 (VDD2), U2.65 (VSS), U2.66 (VSS), U2.67 (VSS), U2.68 (VSS), U2.69 (VSS), U2.70 (VSS), U2.71 (VSS), U2.72 (VSS), U2.73 (VSS), U2.74 (VSS), U2.75 (VSS), U2.76 (VSS), U2.77 (VSS), U2.78 (VSS), U2.79 (VSS), U2.80 (VSS), U2.81 (VSS), U2.82 (VSS), U2.83 (VSS), U2.84 (VSS), U2.85 (VSS), U2.86 (VSS), U2.87 (VSS), U2.88 (VSS), U2.89 (VSS)
- new net JTAG_TCK: U1.40 (DRAM_DQS_C3)
- new net JTAG_TDI: U1.38 (DRAM_DQS_C2)
- new net JTAG_TDO: U1.37 (DRAM_DQS_T2)
- new net JTAG_TMS: U1.39 (DRAM_DQS_T3)
- new net JTAG_TRST_N: U1.36 (DRAM_DQS_C1)
- new net MIPI_CSI0_CLK_N: U1.57 (MIPI_DSI_CLK_P)
- new net MIPI_CSI0_CLK_P: U1.58 (MIPI_DSI_CLK_N)
- new net MIPI_CSI0_D0_N: U1.55 (DRAM_RESET_N)
- new net MIPI_CSI0_D0_P: U1.56 (DRAM_ZQ)
- new net MIPI_CSI0_D1_N: U1.53 (DRAM_CKE)
- new net MIPI_CSI0_D1_P: U1.54 (DRAM_CS)
- new net MIPI_CSI0_D2_N: U1.51 (DRAM_CK_T)
- new net MIPI_CSI0_D2_P: U1.52 (DRAM_CK_C)
- new net MIPI_CSI0_D3_N: U1.49 (DRAM_CA4)
- new net MIPI_CSI0_D3_P: U1.50 (DRAM_CA5)
- new net MIPI_CSI1_CLK_N: U1.47 (DRAM_CA2)
- new net MIPI_CSI1_CLK_P: U1.48 (DRAM_CA3)
- new net MIPI_CSI1_D0_N: U1.45 (DRAM_CA0)
- new net MIPI_CSI1_D0_P: U1.46 (DRAM_CA1)
- new net MIPI_CSI1_D1_N: U1.43 (DRAM_DM2)
- new net MIPI_CSI1_D1_P: U1.44 (DRAM_DM3)
- new net MIPI_DSI_CLK_N: U1.71 (MIPI_CSI0_CLK_P)
- new net MIPI_DSI_CLK_P: U1.72 (MIPI_CSI0_CLK_N)
- new net MIPI_DSI_D0_N: U1.69 (DISP_BL_EN)
- new net MIPI_DSI_D0_P: U1.70 (DISP_BL_PWM)
- new net MIPI_DSI_D1_N: U1.67 (DISP_RESET_N)
- new net MIPI_DSI_D1_P: U1.68 (DISP_TE)
- new net MIPI_DSI_D2_N: U1.65 (MIPI_DSI_D3_P)
- new net MIPI_DSI_D2_P: U1.66 (MIPI_DSI_D3_N)
- new net MIPI_DSI_D3_N: U1.63 (MIPI_DSI_D2_P)
- new net MIPI_DSI_D3_P: U1.64 (MIPI_DSI_D2_N)
- new net OSC_CLK: U1.14 (DRAM_DQ13)
- new net PMIC_I2C_SCL: U1.31 (DRAM_DQ30)
- new net PMIC_I2C_SDA: U1.30 (DRAM_DQ29)
- new net PMIC_IRQ_N: U1.25 (DRAM_DQ24)
- new net PMIC_RESET_N: U1.24 (DRAM_DQ23)
- new net PWR_KEY_N: U1.20 (DRAM_DQ19)
- new net SOC_RESET_N: U1.21 (DRAM_DQ20)
- new net SPMI_SCLK: U1.33 (DRAM_DQS_T0)
- new net SPMI_SDATA: U1.32 (DRAM_DQ31)
- new net UART_RX: U1.34 (DRAM_DQS_C0)
- new net UART_TX: U1.35 (DRAM_DQS_T1)
- new net USBPD_I2C_SCL: U1.29 (DRAM_DQ28)
- new net USBPD_I2C_SDA: U1.28 (DRAM_DQ27)
- new net USBPD_IRQ_N: U1.23 (DRAM_DQ22)
- new net USB_DN: U1.41 (DRAM_DM0)
- new net USB_DP: U1.42 (DRAM_DM1)
- new net VDD2_LPDDR: U1.6 (DRAM_DQ5), U2.90 (VSS), U2.91 (VSS), U2.92 (VSS), U2.93 (VSS)
- new net VDDQ_LPDDR: U1.7 (DRAM_DQ6), U2.94 (VSS), U2.95 (VSS), U2.96 (VSS), U2.97 (VSS)
- new net VDD_CORE: U1.13 (DRAM_DQ12)
- new net VDD_GPU: U1.12 (DRAM_DQ11)
- new net VDD_IO18: U1.10 (DRAM_DQ9)
- new net VDD_IO33: U1.9 (DRAM_DQ8)
- new net VDD_NPU: U1.11 (DRAM_DQ10)
- new net VDD_PLL: U1.8 (DRAM_DQ7)
- new net VOL_DOWN_N: U1.18 (DRAM_DQ17)
- new net VOL_UP_N: U1.19 (DRAM_DQ18)
Other:
- note added: "Compute sheet: E1_PhoneSoC_BGA256 + LPDDR5X_x32 channel-0. DRAM_* nets are 1:1 SoC <-> LPDDR."
- note added: "Decoupling caps are planning placeholders (1 per consolidated rail). Real PI network is owned by power_usb sheet + PDN."
- note removed: "BARO_INT, MAG_INT"
- note removed: "BT_UART_CTS_N, BT_UART_RTS_N, CELL_USB2_DP, CELL_USB2_DN, CELL_PCIE_TX_P, CELL_PCIE_TX_N,"
- note removed: "CAM0_CSI_D2_P, CAM0_CSI_D2_N, CAM0_CSI_D3_P, CAM0_CSI_D3_N, CAM1_CSI_CLK_P, CAM1_CSI_CLK_N,"
- note removed: "CAM1_CSI_D0_P, CAM1_CSI_D0_N, CAM1_CSI_D1_P, CAM1_CSI_D1_N"
- note removed: "CELL_PCIE_RX_P, CELL_PCIE_RX_N"
- note removed: "CODEC_INT, AMP_INT"
- note removed: "DSI_D3_N, DISP_RESET_N, DISP_TE, DISP_BL_EN, DISP_BL_PWM"
- note removed: "LPDDR_DQ2, LPDDR_DQ3, LPDDR_DQS_P, LPDDR_DQS_N, LPDDR_RESET_N, LPDDR_ZQ"
- note removed: "NFC_I2C_SCL, NFC_I2C_SDA, NFC_IRQ_N, NFC_EN, SENSOR_I2C_SCL, SENSOR_I2C_SDA, IMU_INT, ALS_PROX_INT,"
- note removed: "NON-RELEASE SCHEMATIC SKELETON: logical nets only, no ERC/fabrication claim."
- note removed: "SOC_RESET_N"
- note removed: "U_SOC - application_processor - package/e1-demo-pinout.yaml"
- note removed: "audio: I2S_BCLK, I2S_LRCLK, I2S_DOUT, I2S_DIN, PDM_CLK, PDM_DAT, AUDIO_I2C_SCL, AUDIO_I2C_SDA,"
- note removed: "camera: CAM0_CSI_CLK_P, CAM0_CSI_CLK_N, CAM0_CSI_D0_P, CAM0_CSI_D0_N, CAM0_CSI_D1_P, CAM0_CSI_D1_N,"
- note removed: "controls: PWR_KEY_N, VOL_UP_N, VOL_DOWN_N, WIFI_EN, BT_EN, CELL_RESET_N, CELL_W_DISABLE_N, USIM_DET,"
- note removed: "debug_boot: JTAG_TCK, JTAG_TMS, JTAG_TDI, JTAG_TDO, JTAG_TRST_N, BOOT_MODE0, BOOT_MODE1, BOOT_MODE2,"
- note removed: "display: DSI_CLK_P, DSI_CLK_N, DSI_D0_P, DSI_D0_N, DSI_D1_P, DSI_D1_N, DSI_D2_P, DSI_D2_N, DSI_D3_P,"
- note removed: "memory: LPDDR_CK_P, LPDDR_CK_N, LPDDR_CA0, LPDDR_CA1, LPDDR_CA2, LPDDR_CA3, LPDDR_DQ0, LPDDR_DQ1,"
- note removed: "power: AP_0V8, AP_1V1, IO_1V8, GND"
- note removed: "storage: UFS_REFCLK_P, UFS_REFCLK_N, UFS_TX_P, UFS_TX_N, UFS_RX_P, UFS_RX_N, UFS_RESET_N"
- note removed: "usb: USB_DP, USB_DN"
- note removed: "wireless: WIFI_PCIE_TX_P, WIFI_PCIE_TX_N, WIFI_PCIE_RX_P, WIFI_PCIE_RX_N, BT_UART_TX, BT_UART_RX,"
- title: E1 Phone - E1 SoC, Memory, Storage -> E1 Phone - Compute (SoC + LPDDR5X)
