File: packages/chip/board/kicad/e1-phone/schematic/power_usb.kicad_sch (KiCad schematic)
At the start: 0 parts

Commit message: chip(e1-phone): re-render exploded animation with corrected framing + lighting + EGL chunking
Visual self-review of the previous render exposed three defects that this commit closes:

- Camera was at radius 220 mm with 35deg yfov; phone is ~155 mm tall with parts that fly ~150 mm outward at peak explode, so the camera was effectively inside the explosion bubble. Bumped radius to 500 mm and narrowed yfov to 28deg; tilt to 15deg.
- Lights were camera-anchored, so the back of the orange shell went muddy during the 360deg orbit. Switched to world-anchored 3-point lighting.
- pyrender EGL leaked GPU memory and consistently died around frame ~150. Recreating OffscreenRenderer every 30 frames keeps the full 360-frame render stable.

Re-render output (all confirmed by reading 4 keyframes):
- e1-phone-exploded.mp4: 1920x1080, 30 fps, 12 s, h264/yuv420p, 897 KB
- e1-phone-exploded.glb: 98 nodes, 97 meshes, 3 clips (explode/reassemble/turntable), 183 KB
- e1-phone-exploded-frames/: 360 sequential frames + 24 keyframes at 0.5 s

Also restores the chip e1-phone artifacts (mechanical, board, supplier-pinouts, generator scripts) that an out-of-band git reset to origin/develop wiped between my previous commits ae3f83e9e7 / bd0a350198 and the current HEAD.

Co-Authored-By: Claude Opus 4.7 (1M context) <noreply@anthropic.com>
Parts:
- added J1: USB_C_Receptacle, Connector_USB:USB_C_Receptacle_planning, symbol e1_phone:USB_C_24p
- added J2: Battery_4p, Connector:Conn_01x04_planning, symbol e1_phone:Conn_Battery_2p
- added U10: DA9063L, Package_DFN_QFN:QFN-84-1EP_planning, symbol e1_phone:PMIC_DA9063
- added U11: TPS65987DDH, Package_DFN_QFN:QFN-40-1EP_planning, symbol e1_phone:TPS65987DDH
- added U12: MAX77860, Package_DFN_QFN:WLP-28_planning, symbol e1_phone:MAX77860
Connections:
- new net ADCIN1: U11.7 (CC2)
- new net ADCIN2: U11.6 (CC1)
- new net BAT_ID: J2.4 (GND), U12.2 (CHGIN)
- new net BAT_NTC: J2.1 (VBAT), U12.3 (BATT)
- new net BST: U12.28 (VSS)
- new net BUCK1_FB: U10.39 (VSS)
- new net BUCK2_FB: U10.37 (NTC)
- new net BUCK3_FB: U10.35 (ONKEY_N)
- new net BUCK4_FB: U10.33 (RESET_N)
- new net BUCK5_FB: U10.31 (I2C_SDA)
- new net BUCK6_FB: U10.29 (GPIO3)
- new net CHG_I2C_SCL: U12.7 (THM)
- new net CHG_I2C_SDA: U12.6 (ILIM)
- new net CHG_IRQ_N: U12.5 (ICHG)
- new net CHG_OK_N: U12.4 (SYS)
- new net DEBUG1: U11.1 (VIN_3V3)
- new net DEBUG2: U11.40 (VSS)
- new net EN: U12.1 (VBUS)
- new net GND: J1.1 (A1_GND), J1.12 (A12_GND), J1.13 (B1_GND), J1.24 (B12_GND), J2.3 (BAT_ID)
- new net GPIO0: U10.17 (LDO3)
- new net GPIO1: U10.16 (LDO2)
- new net GPIO2: U10.15 (LDO1)
- new net GPIO3: U10.14 (BUCK6_FB)
- new net ICHG: U12.10 (IRQ_N)
- new net ILIM: U12.9 (I2C_SDA)
- new net LDO10: U10.19 (LDO5)
- new net LDO11: U10.18 (LDO4)
- new net LDO3: U10.26 (GPIO0)
- new net LDO4: U10.25 (LDO11)
- new net LDO5: U10.24 (LDO10)
- new net LDO6: U10.23 (LDO9)
- new net LDO7: U10.22 (LDO8)
- new net LDO8: U10.21 (LDO7)
- new net LDO9: U10.20 (LDO6)
- new net LX: U12.27 (VSS)
- new net NTC: U10.6 (BUCK2_FB)
- new net PMIC_I2C_SCL: U10.13 (BUCK6)
- new net PMIC_I2C_SDA: U10.12 (BUCK5_FB)
- new net PMIC_IRQ_N: U10.11 (BUCK5)
- new net PMIC_RESET_N: U10.10 (BUCK4_FB)
- new net PP_HV: U11.17 (SPI_MISO)
- new net PWR_EN: U10.9 (BUCK4)
- new net PWR_KEY_N: U10.8 (BUCK3_FB)
- new net RESET: U11.8 (USB_DP)
- new net SPI_CS_N: U11.2 (VBUS)
- new net SPI_MISO: U11.4 (PP_HV)
- new net SPI_MOSI: U11.3 (VBUS_SENSE)
- new net SPI_SCLK: U11.5 (PP_5V0)
- new net SYS: U10.41 (VSS), U11.16 (SPI_SCLK), U12.11 (CHG_OK_N)
- new net THM: U12.8 (I2C_SCL)
- new net USBPD_I2C_SCL: U11.11 (I2C_SDA)
- new net USBPD_I2C_SDA: U11.10 (I2C_SCL)
- new net USBPD_IRQ_N: U11.9 (USB_DN)
- new net USB_CC1: J1.8 (A8_SBU1), U11.15 (ADCIN2)
- new net USB_CC2: J1.20 (B8_SBU2), U11.14 (ADCIN1)
- new net USB_DN: J1.18 (B6_DP2), J1.6 (A6_DP1), U11.12 (IRQ_N)
- new net USB_DP: J1.19 (B7_DN2), J1.7 (A7_DN1), U11.13 (RESET)
- new net USB_RX1_N: J1.15 (B3_TX2_N)
- new net USB_RX1_P: J1.14 (B2_TX2_P)
- new net USB_RX2_N: J1.3 (A3_TX1_N)
- new net USB_RX2_P: J1.2 (A2_TX1_P)
- new net USB_SBU1: J1.5 (A5_CC1)
- new net USB_SBU2: J1.17 (B5_CC2)
- new net USB_TX1_N: J1.10 (A10_RX2_N)
- new net USB_TX1_P: J1.11 (A11_RX2_P)
- new net USB_TX2_N: J1.22 (B10_RX1_N)
- new net USB_TX2_P: J1.23 (B11_RX1_P)
- new net VBAT: J2.2 (BAT_NTC), U10.42 (VSS), U12.12 (BAT_NTC)
- new net VBUS: J1.16 (B4_VBUS), J1.21 (B9_VBUS), J1.4 (A4_VBUS), J1.9 (A9_VBUS), U11.18 (SPI_MOSI), U11.19 (SPI_CS_N), U12.13 (BAT_ID), U12.14 (EN)
- new net VDD2_LPDDR: U10.30 (I2C_SCL)
- new net VDDQ_LPDDR: U10.32 (IRQ_N)
- new net VDD_CORE: U10.40 (VSS)
- new net VDD_GPU: U10.38 (VSS)
- new net VDD_IO18: U10.34 (PWR_EN)
- new net VDD_IO33: U10.28 (GPIO2), U11.20 (DEBUG1)
- new net VDD_NPU: U10.36 (VREF)
- new net VDD_PLL: U10.27 (GPIO1)
- new net VREF: U10.7 (BUCK3)
- new net VSS: U10.1 (VBAT), U10.2 (VSYS), U10.3 (BUCK1), U10.4 (BUCK1_FB), U10.43 (VSS), U10.44 (VSS), U10.45 (VSS), U10.46 (VSS), U10.47 (VSS), U10.48 (VSS), U10.49 (VSS), U10.5 (BUCK2), U10.50 (VSS), U10.51 (VSS), U10.52 (VSS), U10.53 (VSS), U10.54 (VSS), U10.55 (VSS), U10.56 (VSS), U10.57 (VSS), U10.58 (VSS), U10.59 (VSS), U10.60 (VSS), U10.61 (VSS), U10.62 (VSS), U10.63 (VSS), U10.64 (VSS), U10.65 (VSS), U10.66 (VSS), U10.67 (VSS), U10.68 (VSS), U10.69 (VSS), U10.70 (VSS), U10.71 (VSS), U10.72 (VSS), U10.73 (VSS), U10.74 (VSS), U10.75 (VSS), U10.76 (VSS), U10.77 (VSS), U10.78 (VSS), U10.79 (VSS), U10.80 (VSS), U10.81 (VSS), U10.82 (VSS), U10.83 (VSS), U10.84 (VSS), U11.21 (DEBUG2), U11.22 (VSS), U11.23 (VSS), U11.24 (VSS), U11.25 (VSS), U11.26 (VSS), U11.27 (VSS), U11.28 (VSS), U11.29 (VSS), U11.30 (VSS), U11.31 (VSS), U11.32 (VSS), U11.33 (VSS), U11.34 (VSS), U11.35 (VSS), U11.36 (VSS), U11.37 (VSS), U11.38 (VSS), U11.39 (VSS), U12.15 (BST), U12.16 (LX), U12.17 (VSS), U12.18 (VSS), U12.19 (VSS), U12.20 (VSS), U12.21 (VSS), U12.22 (VSS), U12.23 (VSS), U12.24 (VSS), U12.25 (VSS), U12.26 (VSS)
Other:
- note added: "Power/USB sheet. VBUS -> MAX77860 -> SYS -> DA9063 bucks -> SoC rails. USB-PD CC1/CC2 + USB_DP/DN brought up to root."
- note removed: "J_BATTERY - battery_pack_connector - package/battery/e1-phone-17p3wh-pack.yaml"
- note removed: "J_USB_C - connector - package/usb-c/e1-phone-usb-c-port.yaml"
- note removed: "NON-RELEASE SCHEMATIC SKELETON: logical nets only, no ERC/fabrication claim."
- note removed: "U_CHARGER - charger_power_path - package/charger/max77860.yaml"
- note removed: "U_PMIC - pmic - package/pmic/da9063.yaml"
- note removed: "U_USB_PD - usb_pd_controller - package/usb-pd/tps65987.yaml"
- note removed: "VDD_AMP_3V3"
- note removed: "control: CHG_I2C_SCL, CHG_I2C_SDA, CHG_IRQ_N, BAT_NTC, BAT_ID"
- note removed: "control: PMIC_I2C_SCL, PMIC_I2C_SDA, PMIC_IRQ_N, PMIC_RESET_N, PWR_KEY_N"
- note removed: "control: USB_CC1, USB_CC2"
- note removed: "control: USB_CC1, USB_CC2, USBPD_I2C_SCL, USBPD_I2C_SDA, USBPD_IRQ_N, USBPD_RESET"
- note removed: "esd_required: VBUS, USB_DP, USB_DN, USB_CC1, USB_CC2"
- note removed: "high_speed: USB_DP, USB_DN"
- note removed: "power: VBAT, GND"
- note removed: "power: VBUS, GND, SHIELD_GND"
- note removed: "power: VBUS, VBAT, SYS, GND"
- note removed: "power: VIN_3V3, GND"
- note removed: "power_inputs: SYS, VBAT, GND"
- note removed: "power_outputs: AON_1V8, AP_0V8, AP_1V1, IO_1V8, RF_VBAT, CAM_AVDD_2V8, CAM_DVDD_1V2, VDD_AUDIO_3V3,"
- note removed: "power_path: VBUS"
- note removed: "sense: BAT_NTC, BAT_ID"
- title: E1 Phone - Power, Battery, Charger, USB-C -> E1 Phone - Power, USB-PD, Charger, USB-C, Battery
