Commit message: WIP checkpoint: preserve in-flight TEE/android/robot/os swarm work
Co-Authored-By: Claude Opus 4.7 (1M context) <noreply@anthropic.com>

File: packages/robot/assets/profiles/asimov-1/asimov.urdf (robot description, URDF)
Before this commit: robot asimov-1, 0 links, 0 joints
Links:
- added link left_ankle_pitch_link, mass 0.273090119400173; visual mesh filename=meshes/LEFT_ANKLE_A.STL
- added link left_ankle_roll_link, mass 0.405640437504617; visual mesh filename=meshes/LEFT_ANKLE_B.STL
- added link left_elbow_link, mass 0.662317601299901; visual mesh filename=meshes/LEFT_ELBOW.STL
- added link left_hip_pitch_link, mass 1.05630112217695; visual mesh filename=meshes/LEFT_HIP_PITCH.STL
- added link left_hip_roll_link, mass 0.414368139397033; visual mesh filename=meshes/LEFT_HIP_ROLL.STL
- added link left_hip_yaw_link, mass 1.86657016436158; visual mesh filename=meshes/LEFT_HIP_YAW.STL
- added link left_knee_link, mass 2.39114151033076; visual mesh filename=meshes/LEFT_KNEE.STL
- added link left_shoulder_pitch_link, mass 0.599157136550892; visual mesh filename=meshes/LEFT_SHOULDER_PITCH.STL
- added link left_shoulder_roll_link, mass 1.3132281302001; visual mesh filename=meshes/LEFT_SHOULDER_ROLL.STL
- added link left_shoulder_yaw_link, mass 0.712261755331765; visual mesh filename=meshes/LEFT_SHOULDER_YAW.STL
- added link left_toe_link, mass 0.112221237946844; visual mesh filename=meshes/LEFT_TOE.STL
- added link left_wrist_yaw_link, mass 0.058058790654763; visual mesh filename=meshes/LEFT_WRIST_YAW.STL
- added link neck_pitch_link, mass 0.394055609177456; visual mesh filename=meshes/NECK_PITCH.STL
- added link neck_yaw_link, mass 0.53278930532821; visual mesh filename=meshes/NECK_YAW.STL
- added link pelvis_link, mass 3.50691251175897; visual mesh filename=meshes/IMU_ORIGIN.STL
- added link right_ankle_pitch_link, mass 0.27308917159726; visual mesh filename=meshes/RIGHT_ANKLE_A.STL
- added link right_ankle_roll_link, mass 0.405640437504617; visual mesh filename=meshes/RIGHT_ANKLE_B.STL
- added link right_elbow_link, mass 0.662314258886328; visual mesh filename=meshes/RIGHT_ELBOW.STL
- added link right_hip_pitch_link, mass 1.05629742879001; visual mesh filename=meshes/RIGHT_HIP_PITCH.STL
- added link right_hip_roll_link, mass 0.414825000619808; visual mesh filename=meshes/RIGHT_HIP_ROLL.STL
- added link right_hip_yaw_link, mass 1.86647220449567; visual mesh filename=meshes/RIGHT_HIP_YAW.STL
- added link right_knee_link, mass 2.39110172735043; visual mesh filename=meshes/RIGHT_KNEE.STL
- added link right_shoulder_pitch_link, mass 0.599156105726411; visual mesh filename=meshes/RIGHT_SHOULDER_PITCH.STL
- added link right_shoulder_roll_link, mass 1.31322237625579; visual mesh filename=meshes/RIGHT_SHOULDER_ROLL.STL
- added link right_shoulder_yaw_link, mass 0.712261755331765; visual mesh filename=meshes/RIGHT_SHOULDER_YAW.STL
- added link right_toe_link, mass 0.112221754054884; visual mesh filename=meshes/RIGHT_TOE.STL
- added link right_wrist_yaw_link, mass 0.0580595106779709; visual mesh filename=meshes/RIGHT_WRIST_YAW.STL
- added link waist_yaw_link, mass 8.20850158063177; visual mesh filename=meshes/WAIST_YAW.STL
Joints:
- added joint left_ankle_pitch_joint: type revolute, parent left_knee_link, child left_ankle_pitch_link, origin xyz=0 0 -0.2946623361 rpy=0 0 0, axis 0 1 0, limit lower=-0.35 upper=0.35 effort=20 velocity=20
- added joint left_ankle_roll_joint: type revolute, parent left_ankle_pitch_link, child left_ankle_roll_link, origin xyz=-0.0015 0 -0.009999992 rpy=0 0 0, axis -1 0 0, limit lower=-0.1 upper=0.1 effort=20 velocity=20
- added joint left_elbow_joint: type revolute, parent left_shoulder_yaw_link, child left_elbow_link, origin xyz=0 0 -0.0963013 rpy=0 0 0, axis 0 -1 0, limit lower=0 upper=2.443461 effort=20 velocity=20
- added joint left_hip_pitch_joint: type revolute, parent pelvis_link, child left_hip_pitch_link, origin xyz=-0.052 0.0675 -0.044045 rpy=0 0 0, axis 0 1 0, limit lower=-2.094395 upper=1 effort=20 velocity=20
- added joint left_hip_roll_joint: type revolute, parent left_hip_pitch_link, child left_hip_roll_link, origin xyz=0.0422501 0.04000027594 0 rpy=0 0 0, axis 1 0 0, limit lower=-0.785398 upper=0.785398 effort=20 velocity=20
- added joint left_hip_yaw_joint: type revolute, parent left_hip_roll_link, child left_hip_yaw_link, origin xyz=-0.04225 0 -0.052 rpy=0 0 0, axis 0 0 -1, limit lower=-0.785398 upper=0.785398 effort=20 velocity=20
- added joint left_knee_joint: type revolute, parent left_hip_yaw_link, child left_knee_link, origin xyz=0 0 -0.19564 rpy=0 0 0, axis 0 1 0, limit lower=0 upper=1.5 effort=20 velocity=20
- added joint left_shoulder_pitch_joint: type revolute, parent waist_yaw_link, child left_shoulder_pitch_link, origin xyz=-0.02621282535 0.0965 0.2611404833 rpy=0 0 0, axis 0 1 0, limit lower=-3.141593 upper=0.872665 effort=20 velocity=20
- added joint left_shoulder_roll_joint: type revolute, parent left_shoulder_pitch_link, child left_shoulder_roll_link, origin xyz=0.0001 0.06535322323 0 rpy=0 0 0, axis -1 0 0, limit lower=-1.570796 upper=0 effort=20 velocity=20
- added joint left_shoulder_yaw_joint: type revolute, parent left_shoulder_roll_link, child left_shoulder_yaw_link, origin xyz=0 0 -0.12899875 rpy=0 0 0, axis 0 0 -1, limit lower=-1.570796 upper=1.570796 effort=20 velocity=20
- added joint left_toe_joint: type revolute, parent left_ankle_roll_link, child left_toe_link, origin xyz=0.10253 -0.0043664 -0.0067324 rpy=0 0 0, axis 0.010532 0.99994 0, limit lower=-1.047 upper=0 effort=5 velocity=10
- added joint left_wrist_yaw_joint: type revolute, parent left_elbow_link, child left_wrist_yaw_link, origin xyz=0.08656302208 0 -0.07263499989 rpy=0 0 0, axis 0.7660444431 0 -0.6427876097, limit lower=-3.141593 upper=3.141593 effort=20 velocity=20
- added joint neck_pitch_joint: type revolute, parent neck_yaw_link, child neck_pitch_link, origin xyz=0 0 0.03735 rpy=0 0 0, axis 0 1 0, limit lower=-0.785398 upper=0.785398 effort=20 velocity=20
- added joint neck_yaw_joint: type revolute, parent waist_yaw_link, child neck_yaw_link, origin xyz=-0.01659877455 0 0.3781670296 rpy=0 0 0, axis 0 0 1, limit lower=-1.570796 upper=1.570796 effort=20 velocity=20
- added joint right_ankle_pitch_joint: type revolute, parent right_knee_link, child right_ankle_pitch_link, origin xyz=0 0.0001 -0.2946623361 rpy=0 0 0, axis 0 -1 0, limit lower=-0.35 upper=0.35 effort=20 velocity=20
- added joint right_ankle_roll_joint: type revolute, parent right_ankle_pitch_link, child right_ankle_roll_link, origin xyz=-0.0015 0 -0.009999992 rpy=0 0 0, axis -1 0 0, limit lower=-0.1 upper=0.1 effort=20 velocity=20
- added joint right_elbow_joint: type revolute, parent right_shoulder_yaw_link, child right_elbow_link, origin xyz=0 0 -0.0966013 rpy=0 0 0, axis 0 1 0, limit lower=-2.443461 upper=0 effort=20 velocity=20
- added joint right_hip_pitch_joint: type revolute, parent pelvis_link, child right_hip_pitch_link, origin xyz=-0.052 -0.0675 -0.044045 rpy=0 0 0, axis 0 -1 0, limit lower=-1 upper=2.094395 effort=20 velocity=20
- added joint right_hip_roll_joint: type revolute, parent right_hip_pitch_link, child right_hip_roll_link, origin xyz=0.04225 -0.04 0 rpy=0 0 0, axis 1 0 0, limit lower=-0.785398 upper=0.785398 effort=20 velocity=20
- added joint right_hip_yaw_joint: type revolute, parent right_hip_roll_link, child right_hip_yaw_link, origin xyz=-0.04225 0 -0.052 rpy=0 0 0, axis 0 0 -1, limit lower=-0.785398 upper=0.785398 effort=20 velocity=20
- added joint right_knee_joint: type revolute, parent right_hip_yaw_link, child right_knee_link, origin xyz=0 0 -0.19564 rpy=0 0 0, axis 0 -1 0, limit lower=-1.5 upper=0 effort=20 velocity=20
- added joint right_shoulder_pitch_joint: type revolute, parent waist_yaw_link, child right_shoulder_pitch_link, origin xyz=-0.02621282535 -0.0965 0.2611404833 rpy=0 0 0, axis 0 -1 0, limit lower=-0.872665 upper=3.141593 effort=20 velocity=20
- added joint right_shoulder_roll_joint: type revolute, parent right_shoulder_pitch_link, child right_shoulder_roll_link, origin xyz=0 -0.06535322323 -6.334135041e-05 rpy=0 0 0, axis -1 0 0, limit lower=0 upper=1.570796 effort=20 velocity=20
- added joint right_shoulder_yaw_joint: type revolute, parent right_shoulder_roll_link, child right_shoulder_yaw_link, origin xyz=0 0 -0.12899875 rpy=0 0 0, axis 0 0 -1, limit lower=-1.570796 upper=1.570796 effort=20 velocity=20
- added joint right_toe_joint: type revolute, parent right_ankle_roll_link, child right_toe_link, origin xyz=0.10247 0.0042796 -0.0067324 rpy=0 0 0, axis 0.0074685 -0.99997 0, limit lower=0 upper=1.047 effort=5 velocity=10
- added joint right_wrist_yaw_joint: type revolute, parent right_elbow_link, child right_wrist_yaw_link, origin xyz=0.08656302207 0 -0.07263499989 rpy=0 0 0, axis 0.7660444431 0 -0.6427876097, limit lower=-3.141593 upper=3.141593 effort=20 velocity=20
- added joint waist_yaw_joint: type revolute, parent pelvis_link, child waist_yaw_link, origin xyz=-0.052 0 0.074755 rpy=0 0 0, axis 0 0 1, limit lower=-1.570796 upper=1.570796 effort=20 velocity=20
