File: packages/chip/board/kicad/e1-phone/pcb/e1-phone-mainboard-real-footprint-development.kicad_pcb (KiCad board)
At the start: 10 copper layers, 64 x 132 mm, 89 parts

Commit message: wip: snapshot worktree before pulling latest develop
Concurrent-swarm working-tree state from packages/chip/, packages/os/
evidence, packages/robot/, and upstreams/. Committed (not stashed) per
the repo's git-workflow rule before pulling latest from origin/develop
so nothing is lost across the rebase.

Co-Authored-By: Claude Opus 4.7 (1M context) <noreply@anthropic.com>
Routing:
- added copper zone on B.Cu, net GND
- added copper zone on F.Cu, net GND
- added copper zone on In1.GND, net GND
- added copper zone on In8.GND, net GND
Changed lines of the file:
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@@
   (via (at 8.000 124.000) (size 0.450) (drill 0.200) (layers "F.Cu" "B.Cu") (net 86))
   (via (at 56.000 124.000) (size 0.450) (drill 0.200) (layers "F.Cu" "B.Cu") (net 86))
+  (zone (net 86) (net_name "GND") (layers "F.Cu" "In1.GND" "B.Cu")
+    (name "E1Phone_LOCAL_GND_TOP_ISLAND_POUR")
+    (hatch edge 0.500)
+    (priority 30)
+    (connect_pads (clearance 0.150))
+    (min_thickness 0.100)
+    (fill yes (thermal_gap 0.500) (thermal_bridge_width 0.500))
+    (polygon
+      (pts
+        (xy 1.000 1.000)
+        (xy 63.000 1.000)
+        (xy 63.000 28.200)
+        (xy 1.000 28.200)
+      )
+    )
+  )
+  (zone (net 86) (net_name "GND") (layers "F.Cu" "In8.GND" "B.Cu")
+    (name "E1Phone_LOCAL_GND_BOTTOM_ISLAND_POUR")
+    (hatch edge 0.500)
+    (priority 30)
+    (connect_pads (clearance 0.150))
+    (min_thickness 0.100)
+    (fill yes (thermal_gap 0.500) (thermal_bridge_width 0.500))
+    (polygon
+      (pts
+        (xy 1.000 117.800)
+        (xy 63.000 117.800)
+        (xy 63.000 131.000)
+        (xy 1.000 131.000)
+      )
+    )
+  )
 )
