Commit message: chore: checkpoint generated robot artifacts

File: packages/robot/assets/profiles/erobot/erobot.urdf (robot description, URDF)
Before this commit: robot erobot, 26 links, 25 joints
Links:
- added link left_toe, mass 0.35628; collision box size=0.08 0.1 0.008; collision box size=0.08 0.1 0.045
- added link right_toe, mass 0.35628; collision box size=0.08 0.1 0.008; collision box size=0.08 0.1 0.045
- link left_ankle_pitch: mass 0.52 -> 0.648177; geometry collision sphere radius=0.05; visual sphere radius=0.05
- link left_ankle_roll: mass 1.01764 -> 0.990137; geometry collision box size=0.16 0.1 0.008; collision box size=0.16 0.1 0.045
- link left_elbow: mass 0.732148 -> 0.820898; geometry collision cylinder length=0.26 radius=0.036; collision sphere radius=0.05
- link left_hip_pitch: mass 0.988636 -> 1.03457; geometry collision sphere radius=0.06; visual sphere radius=0.06
- link left_hip_roll: mass 0.978177 -> 1.03457; geometry collision sphere radius=0.06; visual sphere radius=0.06
- link left_knee: mass 1.48494 -> 1.66951; geometry collision cylinder length=0.42 radius=0.048; collision sphere radius=0.06
- link left_wrist_yaw: mass 0.329895 -> 0.398623; geometry collision box size=0.09 0.05 0.17; collision sphere radius=0.044
- link right_ankle_pitch: mass 0.52 -> 0.648177; geometry collision sphere radius=0.05; visual sphere radius=0.05
- link right_ankle_roll: mass 1.01764 -> 0.990137; geometry collision box size=0.16 0.1 0.008; collision box size=0.16 0.1 0.045
- link right_elbow: mass 0.732148 -> 0.820898; geometry collision cylinder length=0.26 radius=0.036; collision sphere radius=0.05
- link right_hip_pitch: mass 0.988636 -> 1.03457; geometry collision sphere radius=0.06; visual sphere radius=0.06
- link right_hip_roll: mass 0.978177 -> 1.03457; geometry collision sphere radius=0.06; visual sphere radius=0.06
- link right_knee: mass 1.48494 -> 1.66951; geometry collision cylinder length=0.42 radius=0.048; collision sphere radius=0.06
- link right_wrist_yaw: mass 0.329895 -> 0.398623; geometry collision box size=0.09 0.05 0.17; collision sphere radius=0.044
Joints:
- added joint left_toe_joint: type revolute, parent left_ankle_roll, child left_toe, origin xyz=0.09 0 -0.0475 rpy=0 0 0, axis 0 1 0, limit lower=-0.6 upper=0.2 effort=10 velocity=12
- added joint right_toe_joint: type revolute, parent right_ankle_roll, child right_toe, origin xyz=0.09 0 -0.0475 rpy=0 0 0, axis 0 1 0, limit lower=-0.6 upper=0.2 effort=10 velocity=12

Commit message: chore: checkpoint concurrent develop fixes

File: packages/robot/assets/profiles/erobot/erobot.urdf (robot description, URDF)
Before this commit: robot erobot, 28 links, 27 joints
Links:
- removed link head
- removed link left_wrist_yaw
- removed link neck
- removed link right_wrist_yaw
- added link spine, mass 0.648177; collision sphere radius=0.05; visual sphere radius=0.05
- link torso: mass 5.94445 -> 6.07262; geometry collision box size=0.19 0.3 0.42; collision sphere radius=0.05
Joints:
- removed joint left_wrist_yaw_joint
- removed joint neck_pitch_joint
- removed joint neck_yaw_joint
- removed joint right_wrist_yaw_joint
- added joint waist_pitch_joint: type revolute, parent spine, child torso, origin xyz=0 0 0.12 rpy=0 0 0, axis 0 1 0, limit lower=-0.5 upper=0.8 effort=24 velocity=20
- joint waist_yaw_joint: child torso -> spine
